File: hardware/n0183to2k.sch (KiCad schematic (older format))
At the start: 34 parts, among them J1 NMEA0183 (wind), J2 Conn_01x06_Male, J3 Conn_01x05_Male, J4 RJ45, J5 RJ45, J6 Conn_02x03_Odd_Even, Q1 BSS123, Q2 DMG2307L, Q3 BSS123, U1 PIC18F27Q84_ISS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

Commit message: Add a LED to a free GPIO.
Parts:
- added D3: red, LED_THT:LED_D3.0mm, symbol Device:LED_Small
- added R10: 330, Resistor_THT:R_Axial_DIN0207_L6.3mm_D2.5mm_P7.62mm_Horizontal, symbol Device:R_Small
Connections:
- net GND: now also R10.1; no longer U1.21 (INT0/RB0)
- new net: D3.2 (A), U1.21 (INT0/RB0)
- new net: D3.1 (K), R10.2
Changed lines of the file:
@@
 L power:GND #PWR06
 U 1 1 6232F043
-P 3650 3800
-F 0 "#PWR06" H 3650 3550 50  0001 C CNN
-F 1 "GND" H 3655 3627 50  0000 C CNN
-F 2 "" H 3650 3800 50  0001 C CNN
-F 3 "" H 3650 3800 50  0001 C CNN
-	1    3650 3800
+P 4050 3850
+F 0 "#PWR06" H 4050 3600 50  0001 C CNN
+F 1 "GND" H 4055 3677 50  0000 C CNN
+F 2 "" H 4050 3850 50  0001 C CNN
+F 3 "" H 4050 3850 50  0001 C CNN
+	1    4050 3850
 	0    -1   -1   0
 $EndComp
 Wire Wire Line
 	3550 3750 3600 3750
-Wire Wire Line
-	3600 3750 3600 3800
-Wire Wire Line
-	3600 3850 3550 3850
-Wire Wire Line
-	3650 3800 3600 3800
-Connection ~ 3600 3800
-Wire Wire Line
-	3600 3800 3600 3850
 Wire Wire Line
 	3550 4150 3600 4150
@@
 	0    -1   -1   0
 $EndComp
+$Comp
+L Device:LED_Small D3
+U 1 1 6221A5B0
+P 3750 3450
+F 0 "D3" H 3750 3243 50  0000 C CNN
+F 1 "red" H 3750 3334 50  0000 C CNN
+F 2 "LED_THT:LED_D3.0mm" V 3750 3450 50  0001 C CNN
+F 3 "~" V 3750 3450 50  0001 C CNN
+	1    3750 3450
+	-1   0    0    1
+$EndComp
+$Comp
+L Device:R_Small R10
+U 1 1 6221BF2C
+P 3950 3550
+F 0 "R10" H 3850 3550 50  0000 C CNN
+F 1 "330" V 4050 3550 50  0000 C CNN
+F 2 "Resistor_THT:R_Axial_DIN0207_L6.3mm_D2.5mm_P7.62mm_Horizontal" H 3950 3550 50  0001 C CNN
+F 3 "~" H 3950 3550 50  0001 C CNN
+	1    3950 3550
+	-1   0    0    1
+$EndComp
+Wire Wire Line
+	3600 3750 3600 3450
+Wire Wire Line
+	3600 3450 3650 3450
+Wire Wire Line
+	3850 3450 3950 3450
+Wire Wire Line
+	3950 3650 3950 3850
+Wire Wire Line
+	3950 3850 4050 3850
+Wire Wire Line
+	3550 3850 3950 3850
+Connection ~ 3950 3850
 $EndSCHEMATC

Commit message: Add mounting holes
Parts:
- added H1, H2, H3, H4: MountingHole, symbol Mechanical:MountingHole
Changed lines of the file:
@@
 	3550 3850 3950 3850
 Connection ~ 3950 3850
+$Comp
+L Mechanical:MountingHole H1
+U 1 1 62257829
+P 6700 4850
+F 0 "H1" H 6800 4896 50  0000 L CNN
+F 1 "MountingHole" H 6800 4805 50  0000 L CNN
+F 2 "" H 6700 4850 50  0001 C CNN
+F 3 "~" H 6700 4850 50  0001 C CNN
+	1    6700 4850
+	1    0    0    -1
+$EndComp
+$Comp
+L Mechanical:MountingHole H2
+U 1 1 62257F08
+P 6700 5050
+F 0 "H2" H 6800 5096 50  0000 L CNN
+F 1 "MountingHole" H 6800 5005 50  0000 L CNN
+F 2 "" H 6700 5050 50  0001 C CNN
+F 3 "~" H 6700 5050 50  0001 C CNN
+	1    6700 5050
+	1    0    0    -1
+$EndComp
+$Comp
+L Mechanical:MountingHole H3
+U 1 1 62258377
+P 6700 5250
+F 0 "H3" H 6800 5296 50  0000 L CNN
+F 1 "MountingHole" H 6800 5205 50  0000 L CNN
+F 2 "" H 6700 5250 50  0001 C CNN
+F 3 "~" H 6700 5250 50  0001 C CNN
+	1    6700 5250
+	1    0    0    -1
+$EndComp
+$Comp
+L Mechanical:MountingHole H4
+U 1 1 6225869C
+P 6700 5450
+F 0 "H4" H 6800 5496 50  0000 L CNN
+F 1 "MountingHole" H 6800 5405 50  0000 L CNN
+F 2 "" H 6700 5450 50  0001 C CNN
+F 3 "~" H 6700 5450 50  0001 C CNN
+	1    6700 5450
+	1    0    0    -1
+$EndComp
 $EndSCHEMATC

Commit message: Add mounting holes
Parts:
- H1, H2, H3, H4: footprint (none) -> MountingHole:MountingHole_3.5mm
Changed lines of the file:
@@
 F 0 "H1" H 6800 4896 50  0000 L CNN
 F 1 "MountingHole" H 6800 4805 50  0000 L CNN
-F 2 "" H 6700 4850 50  0001 C CNN
+F 2 "MountingHole:MountingHole_3.5mm" H 6700 4850 50  0001 C CNN
 F 3 "~" H 6700 4850 50  0001 C CNN
 	1    6700 4850
@@
 F 0 "H2" H 6800 5096 50  0000 L CNN
 F 1 "MountingHole" H 6800 5005 50  0000 L CNN
-F 2 "" H 6700 5050 50  0001 C CNN
+F 2 "MountingHole:MountingHole_3.5mm" H 6700 5050 50  0001 C CNN
 F 3 "~" H 6700 5050 50  0001 C CNN
 	1    6700 5050
@@
 F 0 "H3" H 6800 5296 50  0000 L CNN
 F 1 "MountingHole" H 6800 5205 50  0000 L CNN
-F 2 "" H 6700 5250 50  0001 C CNN
+F 2 "MountingHole:MountingHole_3.5mm" H 6700 5250 50  0001 C CNN
 F 3 "~" H 6700 5250 50  0001 C CNN
 	1    6700 5250
@@
 F 0 "H4" H 6800 5496 50  0000 L CNN
 F 1 "MountingHole" H 6800 5405 50  0000 L CNN
-F 2 "" H 6700 5450 50  0001 C CNN
+F 2 "MountingHole:MountingHole_3.5mm" H 6700 5450 50  0001 C CNN
 F 3 "~" H 6700 5450 50  0001 C CNN
 	1    6700 5450
